File: main_board/main_board.sch (EAGLE design)
At the start: 15 parts, among them Q1 FC-12M, U1 MDBT40SMD, U2 MPU-9250

Commit message: MDBT42
Parts:
- removed C5: .1uF, SparkFun-Capacitors:CAP0603-CAP
- removed U1: MDBT40SMD, MDBT40:MDBT40SMD
- added U$1: MDBT42SMD, MDBT42:MDBT42SMD
- C3: value 1uF -> 10uF
Connections:
- removed net LED4: U1.P0.17
- new net LED0: U$1.P0.20
- new net LED1: U$1.P0.19
- new net NRESET: U$1.P0.21/RESET
- net A0: now also U$1.P0.03; no longer U1.P0.00
- net A1: now also U$1.P0.04; no longer U1.P0.01
- net A2: now also U$1.P0.05; no longer U1.P0.02
- net A3: now also U$1.P0.06; no longer U1.P0.03
- net A4: now also U$1.P0.07; no longer U1.P0.04
- net A5: now also U$1.P0.08; no longer U1.P0.05
- net A6: now also U$1.P0.09; no longer U1.P0.06
- net A7: now also U$1.P0.10; no longer U1.P0.07
- net D0: now also U$1.P0.25; no longer U1.P0.21
- net D1: now also U$1.P0.26; no longer U1.P0.22
- net D2: now also U$1.P0.27; no longer U1.P0.23
- net D3: now also U$1.P0.28; no longer U1.P0.24
- net D4: now also U$1.P0.29; no longer U1.P0.25
- net D5: now also U$1.P0.30; no longer U1.P0.28
- net D6: now also U$1.P0.31; no longer U1.P0.29
- net D7: now also U$1.P0.02; no longer U1.P0.30
- net GND: now also U$1.GND@1, U$1.GND@12, U$1.GND@24, U$1.GND@39; no longer C5.2, U1.GND@1, U1.GND@2, U1.GND@3, U1.GND@4, U1.GND@5
- net N$2: now also U$1.P0.01/XL2; no longer U1.XL2
- net N$3: now also U$1.P0.00/XL1; no longer U1.XL1
- net RX: now also U$1.P0.11; no longer U1.P0.12
- net SPI_MISO: now also U$1.P0.15; no longer U1.P0.14
- net SPI_MOSI: now also U$1.P0.13; no longer U1.P0.09
- net SPI_SCK: now also U$1.P0.14; no longer U1.P0.10
- net SPI_SS: now also U$1.P0.16; no longer U1.P0.15
- net SWCLK: now also J4.2, U$1.SWCLK; no longer J4.3, U1.SWCLK
- net SWDIO: now also J4.3, U$1.SWDIO; no longer J4.2, U1.SWDIO
- net TWI_SCL: now also U$1.P0.18; no longer U1.DEC2
- net TWI_SDA: now also U$1.P0.17; no longer U1.P0.20
- net TX: now also U$1.P0.12; no longer U1.P0.08
- net VCC: now also U$1.VDD; no longer C5.1, U1.AVDD, U1.VDD
Other:
- moved on the sheet: C3, C6, C7, Q1

Commit message: before order r2 board
Parts:
- renumbered U$1 to U1
Changed lines of the file:
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@@
 <part name="GND2" library="SparkFun-Aesthetics" deviceset="GND" device=""/>
 <part name="SUPPLY2" library="SparkFun-Aesthetics" deviceset="VCC" device=""/>
-<part name="U$1" library="MDBT42" deviceset="MDBT42" device="SMD"/>
+<part name="U1" library="MDBT42" deviceset="MDBT42" device="SMD"/>
 </parts>
 <sheets>
@@
 <instance part="GND2" gate="1" x="213.36" y="139.7"/>
 <instance part="SUPPLY2" gate="G$1" x="215.9" y="129.54"/>
-<instance part="U$1" gate="G$1" x="116.84" y="144.78"/>
+<instance part="U1" gate="G$1" x="116.84" y="144.78"/>
 </instances>
 <busses>
@@
 <pinref part="GND4" gate="1" pin="GND"/>
 <wire x1="86.36" y1="167.64" x2="83.82" y2="167.64" width="0.1524" layer="91"/>
-<pinref part="U$1" gate="G$1" pin="GND@1"/>
-<pinref part="U$1" gate="G$1" pin="GND@12"/>
+<pinref part="U1" gate="G$1" pin="GND@1"/>
+<pinref part="U1" gate="G$1" pin="GND@12"/>
 <wire x1="83.82" y1="167.64" x2="71.12" y2="167.64" width="0.1524" layer="91"/>
 <wire x1="101.6" y1="114.3" x2="101.6" y2="111.76" width="0.1524" layer="91"/>
@@
 <segment>
 <pinref part="GND7" gate="1" pin="GND"/>
-<pinref part="U$1" gate="G$1" pin="GND@39"/>
+<pinref part="U1" gate="G$1" pin="GND@39"/>
 <wire x1="147.32" y1="167.64" x2="149.86" y2="167.64" width="0.1524" layer="91"/>
-<pinref part="U$1" gate="G$1" pin="GND@24"/>
+<pinref part="U1" gate="G$1" pin="GND@24"/>
 <wire x1="149.86" y1="167.64" x2="170.18" y2="167.64" width="0.1524" layer="91"/>
 <wire x1="132.08" y1="114.3" x2="132.08" y2="111.76" width="0.1524" layer="91"/>
@@
 <wire x1="50.8" y1="124.46" x2="50.8" y2="127" width="0.1524" layer="91"/>
 <junction x="50.8" y="127"/>
-<pinref part="U$1" gate="G$1" pin="VDD"/>
+<pinref part="U1" gate="G$1" pin="VDD"/>
 <wire x1="50.8" y1="127" x2="86.36" y2="127" width="0.1524" layer="91"/>
 <junction x="50.8" y="127"/>
@@
 <wire x1="147.32" y1="137.16" x2="160.02" y2="137.16" width="0.1524" layer="91"/>
 <label x="152.4" y="137.16" size="2.54" layer="95"/>
-<pinref part="U$1" gate="G$1" pin="P0.16"/>
+<pinref part="U1" gate="G$1" pin="P0.16"/>
 </segment>
 <segment>
@@
 <wire x1="147.32" y1="129.54" x2="160.02" y2="129.54" width="0.1524" layer="91"/>
 <label x="152.4" y="129.54" size="2.54" layer="95"/>
-<pinref part="U$1" gate="G$1" pin="P0.13"/>
+<pinref part="U1" gate="G$1" pin="P0.13"/>
 </segment>
 <segment>
@@
 <wire x1="147.32" y1="132.08" x2="160.02" y2="132.08" width="0.1524" layer="91"/>
 <label x="152.4" y="132.08" size="2.54" layer="95"/>
-<pinref part="U$1" gate="G$1" pin="P0.14"/>
+<pinref part="U1" gate="G$1" pin="P0.14"/>
 </segment>
 <segment>
@@
 <wire x1="147.32" y1="134.62" x2="160.02" y2="134.62" width="0.1524" layer="91"/>
 <label x="152.4" y="134.62" size="2.54" layer="95"/>
-<pinref part="U$1" gate="G$1" pin="P0.15"/>
+<pinref part="U1" gate="G$1" pin="P0.15"/>
 </segment>
 <segment>
@@
 <junction x="68.58" y="104.14"/>
 <wire x1="68.58" y1="104.14" x2="81.28" y2="104.14" width="0.1524" layer="91"/>
-<pinref part="U$1" gate="G$1" pin="P0.01/XL2"/>
+<pinref part="U1" gate="G$1" pin="P0.01/XL2"/>
 <wire x1="81.28" y1="104.14" x2="106.68" y2="104.14" width="0.1524" layer="91"/>
 <wire x1="106.68" y1="104.14" x2="106.68" y2="114.3" width="0.1524" layer="91"/>
@@
 <junction x="68.58" y="109.22"/>
 <wire x1="68.58" y1="109.22" x2="81.28" y2="109.22" width="0.1524" layer="91"/>
-<pinref part="U$1" gate="G$1" pin="P0.00/XL1"/>
+<pinref part="U1" gate="G$1" pin="P0.00/XL1"/>
 <wire x1="104.14" y1="109.22" x2="104.14" y2="114.3" width="0.1524" layer="91"/>
 </segment>
@@
 <wire x1="147.32" y1="127" x2="160.02" y2="127" width="0.1524" layer="91"/>
 <label x="152.4" y="127" size="2.54" layer="95"/>
-<pinref part="U$1" gate="G$1" pin="P0.12"/>
+<pinref part="U1" gate="G$1" pin="P0.12"/>
 </segment>
 </net>
@@
 <wire x1="147.32" y1="124.46" x2="160.02" y2="124.46" width="0.1524" layer="91"/>
 <label x="152.4" y="124.46" size="2.54" layer="95"/>
-<pinref part="U$1" gate="G$1" pin="P0.11"/>
+<pinref part="U1" gate="G$1" pin="P0.11"/>
 </segment>
 </net>
@@
 <wire x1="129.54" y1="114.3" x2="129.54" y2="104.14" width="0.1524" layer="91"/>
 <label x="129.54" y="104.14" size="2.54" layer="95" rot="R90"/>
-<pinref part="U$1" gate="G$1" pin="P0.10"/>
+<pinref part="U1" gate="G$1" pin="P0.10"/>
 </segment>
 </net>
@@
 <wire x1="127" y1="114.3" x2="127" y2="104.14" width="0.1524" layer="91"/>
 <label x="127" y="104.14" size="2.54" layer="95" rot="R90"/>
-<pinref part="U$1" gate="G$1" pin="P0.09"/>
+<pinref part="U1" gate="G$1" pin="P0.09"/>
 </segment>
 </net>
@@
 <wire x1="124.46" y1="114.3" x2="124.46" y2="104.14" width="0.1524" layer="91"/>
 <label x="124.46" y="104.14" size="2.54" layer="95" rot="R90"/>
-<pinref part="U$1" gate="G$1" pin="P0.08"/>
+<pinref part="U1" gate="G$1" pin="P0.08"/>
 </segment>
 </net>
@@
 <wire x1="121.92" y1="114.3" x2="121.92" y2="104.14" width="0.1524" layer="91"/>
 <label x="121.92" y="104.14" size="2.54" layer="95" rot="R90"/>
-<pinref part="U$1" gate="G$1" pin="P0.07"/>
+<pinref part="U1" gate="G$1" pin="P0.07"/>
 </segment>
 </net>
@@
 <wire x1="119.38" y1="114.3" x2="119.38" y2="104.14" width="0.1524" layer="91"/>
 <label x="119.38" y="104.14" size="2.54" layer="95" rot="R90"/>
-<pinref part="U$1" gate="G$1" pin="P0.06"/>
+<pinref part="U1" gate="G$1" pin="P0.06"/>
 </segment>
 </net>
@@
 <wire x1="116.84" y1="114.3" x2="116.84" y2="104.14" width="0.1524" layer="91"/>
 <label x="116.84" y="104.14" size="2.54" layer="95" rot="R90"/>
-<pinref part="U$1" gate="G$1" pin="P0.05"/>
+<pinref part="U1" gate="G$1" pin="P0.05"/>
 </segment>
 </net>
@@
 <wire x1="114.3" y1="114.3" x2="114.3" y2="104.14" width="0.1524" layer="91"/>
 <label x="114.3" y="104.14" size="2.54" layer="95" rot="R90"/>
-<pinref part="U$1" gate="G$1" pin="P0.04"/>
+<pinref part="U1" gate="G$1" pin="P0.04"/>
 </segment>
 </net>
@@
 <wire x1="111.76" y1="114.3" x2="111.76" y2="104.14" width="0.1524" layer="91"/>
 <label x="111.76" y="104.14" size="2.54" layer="95" rot="R90"/>
-<pinref part="U$1" gate="G$1" pin="P0.03"/>
+<pinref part="U1" gate="G$1" pin="P0.03"/>
 </segment>
 </net>
@@
 <wire x1="109.22" y1="114.3" x2="109.22" y2="104.14" width="0.1524" layer="91"/>
 <label x="109.22" y="104.14" size="2.54" layer="95" rot="R90"/>
-<pinref part="U$1" gate="G$1" pin="P0.02"/>
+<pinref part="U1" gate="G$1" pin="P0.02"/>
 </segment>
 </net>
@@
 <wire x1="86.36" y1="134.62" x2="76.2" y2="134.62" width="0.1524" layer="91"/>
 <label x="76.2" y="134.62" size="2.54" layer="95"/>
-<pinref part="U$1" gate="G$1" pin="P0.31"/>
+<pinref part="U1" gate="G$1" pin="P0.31"/>
 </segment>
 </net>
@@
 <wire x1="86.36" y1="137.16" x2="76.2" y2="137.16" width="0.1524" layer="91"/>
 <label x="76.2" y="137.16" size="2.54" layer="95"/>
-<pinref part="U$1" gate="G$1" pin="P0.30"/>
+<pinref part="U1" gate="G$1" pin="P0.30"/>
 </segment>
 </net>
@@
 <wire x1="86.36" y1="139.7" x2="76.2" y2="139.7" width="0.1524" layer="91"/>
 <label x="76.2" y="139.7" size="2.54" layer="95"/>
-<pinref part="U$1" gate="G$1" pin="P0.29"/>
+<pinref part="U1" gate="G$1" pin="P0.29"/>
 </segment>
 </net>
@@
 <wire x1="86.36" y1="142.24" x2="76.2" y2="142.24" width="0.1524" layer="91"/>
 <label x="76.2" y="142.24" size="2.54" layer="95"/>
-<pinref part="U$1" gate="G$1" pin="P0.28"/>
+<pinref part="U1" gate="G$1" pin="P0.28"/>
 </segment>
 </net>
@@
 <wire x1="86.36" y1="144.78" x2="76.2" y2="144.78" width="0.1524" layer="91"/>
 <label x="76.2" y="144.78" size="2.54" layer="95"/>
-<pinref part="U$1" gate="G$1" pin="P0.27"/>
+<pinref part="U1" gate="G$1" pin="P0.27"/>
 </segment>
 </net>
@@
 <wire x1="86.36" y1="147.32" x2="76.2" y2="147.32" width="0.1524" layer="91"/>
 <label x="76.2" y="147.32" size="2.54" layer="95"/>
-<pinref part="U$1" gate="G$1" pin="P0.26"/>
+<pinref part="U1" gate="G$1" pin="P0.26"/>
 </segment>
 </net>
@@
 <wire x1="86.36" y1="149.86" x2="76.2" y2="149.86" width="0.1524" layer="91"/>
 <label x="76.2" y="149.86" size="2.54" layer="95"/>
-<pinref part="U$1" gate="G$1" pin="P0.25"/>
+<pinref part="U1" gate="G$1" pin="P0.25"/>
 </segment>
 </net>
@@
 <segment>
 <label x="152.4" y="147.32" size="2.54" layer="95"/>
-<pinref part="U$1" gate="G$1" pin="P0.20"/>
+<pinref part="U1" gate="G$1" pin="P0.20"/>
 <wire x1="147.32" y1="147.32" x2="160.02" y2="147.32" width="0.1524" layer="91"/>
 </segment>
@@
 <wire x1="147.32" y1="152.4" x2="160.02" y2="152.4" width="0.1524" layer="91"/>
 <label x="152.4" y="152.4" size="2.54" layer="95"/>
-<pinref part="U$1" gate="G$1" pin="SWCLK"/>
+<pinref part="U1" gate="G$1" pin="SWCLK"/>
 </segment>
 <segment>
@@
 <wire x1="147.32" y1="154.94" x2="160.02" y2="154.94" width="0.1524" layer="91"/>
 <label x="152.4" y="154.94" size="2.54" layer="95"/>
-<pinref part="U$1" gate="G$1" pin="SWDIO"/>
+<pinref part="U1" gate="G$1" pin="SWDIO"/>
 </segment>
 <segment>
@@
 <wire x1="147.32" y1="142.24" x2="160.02" y2="142.24" width="0.1524" layer="91"/>
 <label x="152.4" y="142.24" size="2.54" layer="95"/>
-<pinref part="U$1" gate="G$1" pin="P0.18"/>
+<pinref part="U1" gate="G$1" pin="P0.18"/>
 </segment>
 <segment>
@@
 <wire x1="147.32" y1="139.7" x2="160.02" y2="139.7" width="0.1524" layer="91"/>
 <label x="152.4" y="139.7" size="2.54" layer="95"/>
-<pinref part="U$1" gate="G$1" pin="P0.17"/>
+<pinref part="U1" gate="G$1" pin="P0.17"/>
 </segment>
 <segment>
@@
 <net name="NRESET" class="0">
 <segment>
-<pinref part="U$1" gate="G$1" pin="P0.21/RESET"/>
+<pinref part="U1" gate="G$1" pin="P0.21/RESET"/>
 <wire x1="147.32" y1="149.86" x2="160.02" y2="149.86" width="0.1524" layer="91"/>
 <label x="152.4" y="149.86" size="2.54" layer="95"/>
@@
 <net name="LED1" class="0">
 <segment>
-<pinref part="U$1" gate="G$1" pin="P0.19"/>
+<pinref part="U1" gate="G$1" pin="P0.19"/>
 <wire x1="147.32" y1="144.78" x2="160.02" y2="144.78" width="0.1524" layer="91"/>
 <label x="152.4" y="144.78" size="2.54" layer="95"/>
