File: production_board/merge.sch (EAGLE design)
At the start: 57 parts, among them Q1 FC-12M, Q2 FC-12M, Q3 FC-12M, U1 MDBT40SMD, U2 MPU-9250, U3 MDBT40SMD, U4 MPU-9250, U5 MDBT40SMD, U6 MPU-9250

Commit message: before order r2 board
Parts:
- removed C13, C15: 1uF, SparkFun-Capacitors:CAP0603-CAP
- removed C14: .1uF, SparkFun-Capacitors:CAP0603-CAP
- C10: value 1uF -> 12pF
- C11: value 12pF -> 10uF
- C12: value 12pF -> 1uF
- C3: value 1uF -> 10uF
- C5: value .1uF -> 10uF
- C9: value .1uF -> 12pF
- U1: value MDBT40SMD -> MDBT42SMD; device MDBT40:MDBT40SMD -> MDBT42:MDBT42SMD
- U3, U5: value MDBT40SMD -> MPU-9250; device MDBT40:MDBT40SMD -> invensense:MPU-9250
- U4, U6: value MPU-9250 -> MDBT42SMD; device invensense:MPU-9250 -> MDBT42:MDBT42SMD
Connections:
- removed net LED4: U1.P0.17, U3.P0.17, U5.P0.17
- removed net N$1: C2.1, Q2.1, U3.XL2
- removed net N$10: C4.1, Q2.2, U3.XL1
- removed net N$11: C10.2, U4.REGOUT
- removed net N$17: C11.1, Q3.1, U5.XL2
- removed net N$18: C12.1, Q3.2, U5.XL1
- removed net N$19: C15.2, U6.REGOUT
- new net LED0: U1.P0.20, U4.P0.20, U6.P0.20
- new net LED1: U1.P0.19, U4.P0.19, U6.P0.19
- new net N$100: C4.1, Q2.2, U4.P0.00/XL1
- new net N$101: C8.2, U3.REGOUT
- new net N$107: C9.1, Q3.1, U6.P0.01/XL2
- new net N$108: C10.1, Q3.2, U6.P0.00/XL1
- new net N$109: C12.2, U5.REGOUT
- new net N$64: C2.1, Q2.1, U4.P0.01/XL2
- new net NRESET: U1.P0.21/RESET, U4.P0.21/RESET, U6.P0.21/RESET
- net A0: now also U1.P0.03, U4.P0.03, U6.P0.03; no longer U1.P0.00, U3.P0.00, U5.P0.00
- net A1: now also U1.P0.04, U4.P0.04, U6.P0.04; no longer U1.P0.01, U3.P0.01, U5.P0.01
- net A2: now also U1.P0.05, U4.P0.05, U6.P0.05; no longer U1.P0.02, U3.P0.02, U5.P0.02
- net A3: now also U1.P0.06, U4.P0.06, U6.P0.06; no longer U1.P0.03, U3.P0.03, U5.P0.03
- net A4: now also U1.P0.07, U4.P0.07, U6.P0.07; no longer U1.P0.04, U3.P0.04, U5.P0.04
- net A5: now also U1.P0.08, U4.P0.08, U6.P0.08; no longer U1.P0.05, U3.P0.05, U5.P0.05
- net A6: now also U1.P0.09, U4.P0.09, U6.P0.09; no longer U1.P0.06, U3.P0.06, U5.P0.06
- net A7: now also U1.P0.10, U4.P0.10, U6.P0.10; no longer U1.P0.07, U3.P0.07, U5.P0.07
- net D0: now also U1.P0.25, U4.P0.25, U6.P0.25; no longer U1.P0.21, U3.P0.21, U5.P0.21
- net D1: now also U1.P0.26, U4.P0.26, U6.P0.26; no longer U1.P0.22, U3.P0.22, U5.P0.22
- net D2: now also U1.P0.27, U4.P0.27, U6.P0.27; no longer U1.P0.23, U3.P0.23, U5.P0.23
- net D3: now also U1.P0.28, U4.P0.28, U6.P0.28; no longer U1.P0.24, U3.P0.24, U5.P0.24
- net D4: now also U1.P0.29, U4.P0.29, U6.P0.29; no longer U1.P0.25, U3.P0.25, U5.P0.25
- net D5: now also U1.P0.30, U4.P0.30, U6.P0.30; no longer U1.P0.28, U3.P0.28, U5.P0.28
- net D6: now also U1.P0.31, U4.P0.31, U6.P0.31; no longer U1.P0.29, U3.P0.29, U5.P0.29
- net D7: now also U1.P0.02, U4.P0.02, U6.P0.02; no longer U1.P0.30, U3.P0.30, U5.P0.30
- net GND: now also C10.2, C12.1, C8.1, U1.GND@12, U1.GND@24, U1.GND@39, U3.ADO/SDO, U3.FSYNC, U3.GND, U3.RESV2, U4.GND@1, U4.GND@12, U4.GND@24, U4.GND@39, U5.ADO/SDO, U5.FSYNC, U5.GND, U5.RESV2, U6.GND@1, U6.GND@12, U6.GND@24, U6.GND@39; no longer C10.1, C12.2, C13.2, C14.2, C15.1, C8.2, U1.GND@2, U1.GND@3, U1.GND@4, U1.GND@5, U3.GND@1, U3.GND@2, U3.GND@3, U3.GND@4, U3.GND@5, U4.ADO/SDO, U4.FSYNC, U4.GND, U4.RESV2, U5.GND@1, U5.GND@2, U5.GND@3, U5.GND@4, U5.GND@5, U6.ADO/SDO, U6.FSYNC, U6.GND, U6.RESV2
- net N$2: now also U1.P0.01/XL2; no longer U1.XL2
- net N$3: now also U1.P0.00/XL1; no longer U1.XL1
- net RX: now also U1.P0.11, U4.P0.11, U6.P0.11; no longer U1.P0.12, U3.P0.12, U5.P0.12
- net SPI_MISO: now also U1.P0.15, U4.P0.15, U6.P0.15; no longer U1.P0.14, U3.P0.14, U5.P0.14
- net SPI_MOSI: now also U1.P0.13, U4.P0.13, U6.P0.13; no longer U1.P0.09, U3.P0.09, U5.P0.09
- net SPI_SCK: now also U1.P0.14, U4.P0.14, U6.P0.14; no longer U1.P0.10, U3.P0.10, U5.P0.10
- net SPI_SS: now also U1.P0.16, U4.P0.16, U6.P0.16; no longer U1.P0.15, U3.P0.15, U5.P0.15
- net SWCLK: now also J11.2, J18.2, J4.2, U4.SWCLK, U6.SWCLK; no longer J11.3, J18.3, J4.3, U3.SWCLK, U5.SWCLK
- net SWDIO: now also J11.3, J18.3, J4.3, U4.SWDIO, U6.SWDIO; no longer J11.2, J18.2, J4.2, U3.SWDIO, U5.SWDIO
- net TWI_SCL: now also U1.P0.18, U3.SCL/SCLK, U4.P0.18, U5.SCL/SCLK, U6.P0.18; no longer U1.DEC2, U3.DEC2, U4.SCL/SCLK, U5.DEC2, U6.SCL/SCLK
- net TWI_SDA: now also U1.P0.17, U3.SDA/SDI, U4.P0.17, U5.SDA/SDI, U6.P0.17; no longer U1.P0.20, U3.P0.20, U4.SDA/SDI, U5.P0.20, U6.SDA/SDI
- net TX: now also U1.P0.12, U4.P0.12, U6.P0.12; no longer U1.P0.08, U3.P0.08, U5.P0.08
- net VCC: now also C11.1, U3.NCS, U3.RESV, U3.VDDIO, U5.NCS, U5.RESV, U5.VDDIO; no longer C13.1, C14.1, C8.1, C9.1, U1.AVDD, U3.AVDD, U4.NCS, U4.RESV, U4.VDDIO, U5.AVDD, U6.NCS, U6.RESV, U6.VDDIO
