File: spacer_board/spacer_board.brd (EAGLE design)
At the start: 32.5 x 32.5 mm, 7 parts

Commit message: before order r2 board
Parts:
- moved U$3 20.1 mm to (12.3, 7.24), turned to 0 degrees
Other:
- outline, holes or cut-outs redrawn
Changed lines of the file:
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@@
 <wire x1="15.7242" y1="3.567159375" x2="16.522" y2="3.5588" width="0.001" layer="20"/>
 <wire x1="16.522" y1="3.5588" x2="17.3187" y2="3.600540625" width="0.001" layer="20"/>
-<wire x1="10.756" y1="5.756" x2="21.756" y2="5.756" width="0.001" layer="20"/>
-<wire x1="21.756" y1="5.756" x2="21.756" y2="24.756" width="0.001" layer="20"/>
-<wire x1="21.756" y1="24.756" x2="10.756" y2="24.756" width="0.001" layer="20"/>
-<wire x1="10.756" y1="24.756" x2="10.756" y2="5.756" width="0.001" layer="20"/>
+<wire x1="10.756" y1="8.677" x2="21.756" y2="8.677" width="0.001" layer="20"/>
+<wire x1="21.756" y1="8.677" x2="21.756" y2="23.74" width="0.001" layer="20"/>
+<wire x1="21.756" y1="23.74" x2="10.756" y2="23.74" width="0.001" layer="20"/>
+<wire x1="10.756" y1="23.74" x2="10.756" y2="8.677" width="0.001" layer="20"/>
 </plain>
 <attributes>
@@
 <attribute name="VALUE" x="28.92075" y="11.10475" size="1.27" layer="27" rot="R90"/>
 </element>
-<element name="U$3" library="SparkFun-Connectors_2" package="1X04_HOLE" value="" x="20.066" y="25.781" smashed="yes" rot="R180">
-<attribute name="NAME" x="21.4122" y="23.9522" size="1.27" layer="25" ratio="10" rot="R180" display="off"/>
-<attribute name="VALUE" x="21.336" y="28.956" size="1.27" layer="27" rot="R180"/>
+<element name="U$3" library="SparkFun-Connectors_2" package="1X04_HOLE" value="" x="12.319" y="7.239" smashed="yes">
+<attribute name="NAME" x="10.9728" y="9.0678" size="1.27" layer="25" ratio="10" display="off"/>
+<attribute name="VALUE" x="11.049" y="4.064" size="1.27" layer="27"/>
 </element>
 <element name="U$4" library="SparkFun-Connectors_2" package="1X08_HOLE" value="" x="23.19625" y="7.29875" smashed="yes" rot="R90">
